File: hardware/pcb/badge.kicad_pcb (KiCad board)
At the start: 2 copper layers, 91 x 84 mm, 57 parts, among them J1 EPD FPC 24P 0.5mm, J2 BATT JST-SH 1.0mm, J3 USB-C 16P 沉板 (TYPE-C-31-M-14), Q1 AO3400A, Q2 AO3401A, SW1 RESET, SW2 BOOT/USER, U1 ESP32-C3-MINI-1-N4, U2 ST25DV64KC-IER6S3, U3 TP4054 / MCP73831T-2ACI/OT, U4 XC6220B331MR-G

Commit message: Route PCB (Freerouting + GND stitching), add enclosure, BOM, firmware pin map, export script
Co-authored-by: kongm3270 <kongm3270@outlook.com>
Parts:
- moved C8 12.7 mm to (51.5, 48.8)
- moved R7 7.10 mm to (51.5, 51.4)
- moved C6 4.10 mm to (51.5, 56.6)
- moved C14 3.50 mm to (42.0, 64.5)
- moved J1 3.00 mm to (40.0, 73.0)
- moved C7 1.50 mm to (51.5, 54.0)
- moved SW2 1.50 mm to (22.5, 80.5)
Routing:
- net +3V3: track 0.00 -> 174.1 mm, vias 0 -> 9
- net VBAT: track 0.00 -> 118.7 mm, vias 0 -> 2
- net BOOT_n: track 0.00 -> 94.3 mm, vias 0 -> 2
- net EN: track 0.00 -> 87.2 mm, vias 0 -> 2
- net EPD_CS: track 0.00 -> 74.3 mm, vias 0 -> 2
- net EPD_MOSI: track 0.00 -> 52.5 mm, vias 0 -> 4
- net LED_STAT_n: track 0.00 -> 50.7 mm, vias 0 -> 4
- net EPD_VCI: track 0.00 -> 43.9 mm, vias 0 -> 4
- net EPD_SCK: track 0.00 -> 39.9 mm, vias 0 -> 2
- net EPD_DC: track 0.00 -> 39.2 mm, vias 0 -> 2
- net EPD_RST: track 0.00 -> 39.0 mm, vias 0 -> 2
- net EPD_PWR_EN: track 0.00 -> 38.6 mm, vias 0 -> 4
- net NFC_GPO: track 0.00 -> 35.6 mm, vias 0 -> 3
- net USB_DN: track 0.00 -> 35.1 mm, vias 0 -> 2
- net EPD_GDR: track 0.00 -> 31.9 mm, vias 0 -> 2
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Other:
- outline, holes or cut-outs redrawn

Commit message: Stitch GND pour islands to DRC-clean PCB and write handoff for next session
Current board is 564 tracks / 128 vias with zero DRC errors. route_pcb.py
gains island stitching, J1 pin 7 to GND, ESP GND net-tie, and via nudge.
Handoff and review checklist capture remaining work: make stitching
reproducible, NFC soldermask, fab review, firmware.

Co-authored-by: kongm3270 <kongm3270@outlook.com>
Connections:
- J1 pad 7: (no net) -> GND
Routing:
- net GND: track 0.00 -> 8.30 mm, vias 0 -> 50
