File: hardware/pcb/badge.kicad_sch (KiCad schematic)
At the start: 57 parts, among them J1 EPD FPC 24P 0.5mm, J2 BATT JST-SH 1.0mm, J3 USB-C 16P 沉板 (TYPE-C-31-M-14), Q1 AO3400A, Q2 AO3401A, SW1 RESET, SW2 BOOT/USER, U1 ESP32-C3-MINI-1-N4, U2 ST25DV64KC-IER6S3, U3 TP4054 / MCP73831T-2ACI/OT, U4 XC6220B331MR-G

Commit message: Land H2 board (KiCad 10 full ERC/DRC 0) and firmware v0.2 F1.
Freeze the 680/115 board, hygiene scripts, and self-test fixes (GPIO1 wake, serial W, BUSY fail-closed) so GitHub matches the local pass. v0.1 bins stay as baseline.

Co-authored-by: Cursor <cursoragent@cursor.com>
Parts:
- removed U2: ST25DV64KC-IER6S3, Package_SO:SOIC-8_3.9x4.9mm_P1.27mm, symbol RF_NFC:ST25DV64K-IER8C3
- added R15: 1M, Resistor_SMD:R_0402_1005Metric, symbol Device:R
- added U2: ST25DV64KC-IER6S3, Package_SO:SOIC-8_3.9x4.9mm_P1.27mm, symbol Badge:ST25DV64KC-SO8N
- ANT1, TP1, TP2, TP3, TP4: now left out of the parts list
- C15: value 1u/50V -> 4.7u/25V
- C3: value 1u -> 10u; footprint Capacitor_SMD:C_0402_1005Metric -> Capacitor_SMD:C_0603_1608Metric
- C4: value 2.2u -> 4.7u
- J2: value BATT JST-SH 1.0mm -> BATT JST-SHL 1.0mm; footprint Connector_JST:JST_SHL_SM02B-SHLS-TF_1x02-1MP_P1.00mm_Horizontal -> badge:JST_SHL_SM02B-SHLS-TF_1x02-1MP_P1.00mm_Horizontal
- L1: value 68uH -> 47uH; footprint Inductor_SMD:L_Changjiang_FNR3015S -> Inductor_SMD:L_Changjiang_FNR4018S; LCSC C2827366 -> C167813
- Q1: value AO3400A -> Si1308EDL; footprint Package_TO_SOT_SMD:SOT-23 -> badge:SOT-323_SC-70; LCSC C20917 -> C469327
- R14: footprint Resistor_SMD:R_0402_1005Metric -> Resistor_SMD:R_0603_1608Metric
- U3: value TP4054 / MCP73831T-2ACI/OT -> TP4054
Connections:
- net +3V3: now also U2.8 (VCC)
- net EPD_GDR: now also R15.1
- net GND: now also J3.SH (SHIELD), R15.2, U2.4 (VSS); no longer J1.7 (Pin_7), J3.S1 (SHIELD)
- net I2C_SCL: now also U2.6 (SCL)
- net I2C_SDA: now also U2.5 (SDA)
- net NFC_AC0: now also U2.2 (AC0)
- net NFC_AC1: now also U2.3 (AC1)
- net NFC_GPO: now also U2.7 (GPO)
- net NFC_VEH: now also U2.1 (V_EH)
- no-connect marks 21 -> 22
Other:
- note added: "EPD - 4.2" BWRY GDEM042F86. Boost per p.29: 47uH/500mA-class (FNR4018S470MT 700mA Isat), Si1308EDL, 4.7uF flying cap, GDR 1M to GND, RESE 2.2R 0603. Pin 7 NC Keep Open (p.7). BS1=GND -> 4-wire SPI. Panel power gated by Q2."
- note added: "POWER - LiPo 202545 250mAh 2.0mm with PCM, J2-1=VBAT. TP4054 ~200mA. XC6220 near-end CIN=10uF CL=4.7uF. Standby current is unmeasured; do not quote 13uA or two years."
- note removed: "EPD - 4.2" BWRY panel, 24P 0.5mm FPC (GDEM042F86 / Waveshare 4.2 G / GDEY042F51). Standard Good Display boost: 68uH, N-MOS, 3x MBR0530, RESE. BS1=GND -> 4-wire SPI. VDDIO tied to VCI. Panel power gated by Q2."
- note removed: "POWER - LiPo (<=2.0mm, 150-300mAh, with PCM) -> 200mA linear charger -> low-Iq LDO 3.3V. VBAT sensed through 1M/1M (ADC1_CH0). Standby budget ~13uA."
